Commit message: Remove code-sections related to calibration file.

File: config/bno08x.urdf.xacro (robot description, xacro)
@@ -11,6 +11,4 @@
   <xacro:arg name="enable_mock_mode" default="false"/>
   <xacro:arg name="sensor_mode"      default="NDOF"/>  <!-- Fusion mode: NDOF, NDOF_FMC_OFF, IMUPLUS (default: NDOF) -->
-  <xacro:arg name="calib_file"       default=""/>      <!-- Path to calibration YAML file (empty = uncalibrated startup) -->
-  <xacro:property name="calib_file_path" value="$(arg calib_file)"/>
   <!-- Robot links -->
   <link name="base_link"/>
@@ -44,7 +42,4 @@
       <param name="sensor_mode">$(arg sensor_mode)</param>   <!-- Fusion mode: NDOF, NDOF_FMC_OFF, IMUPLUS (default: NDOF) -->
       <param name="enable_mock_mode">$(arg enable_mock_mode)</param>   <!-- Simulation mode, no hardware required (default: false) -->
-      <xacro:if value="${calib_file_path != ''}">             <!-- Only emitted when a path is provided -->
-        <param name="calib_file">${calib_file_path}</param>
-      </xacro:if>
     </hardware>
     <sensor name="bno08x">
